File: Eagle_Verzeichnisse/Projekte/Matrix-Konsole/controller.sch (EAGLE design)
At the start: 20 parts, among them IC1 74HC165D

Commit message: Changed the matrix board
Parts:
- C1, C2, C3, C4, C5, C6: value (none) -> 100n
- R1, R2, R3, R4, R5, R6: device resistor:R-EU_0414/5V -> resistor:R-EU_M3516
Connections:
- net VCC renamed 5V
