File: Eagle_Verzeichnisse/Projekte/Matrix-Konsole/console.sch (EAGLE design)
At the start: 15 parts, among them J1 DIN5, J2 DIN5, J3 DIN5, J4 DIN5, X2 057-016-1

Commit message: Splitted the console-layout into three boards and improved the layouts
Parts:
- removed 7SEG1, 7SEG2: 7SEG_DEV, seven_segment:7SEG_DEV
- removed C1: 100n, eagle-ltspice:C
- removed J1, J2, J3, J4: DIN5, SparkFun-Connectors:DIN5
- removed R1: 200, resistor:R-EU_M3516
- removed U$2: MAX7219CWG, max7219:MAX7219CWG
- added JP3: (no value), pinhead:PINHD-1X5
- added JP4: (no value), pinhead:PINHD-1X4
- JP2: device pinhead:PINHD-1X4 -> pinhead:PINHD-1X8
Connections:
- removed net A: 7SEG1.A, 7SEG2.A, U$2.SEGA
- removed net B: 7SEG1.B, 7SEG2.B, U$2.SEGB
- removed net C: 7SEG1.C, 7SEG2.C, U$2.SEGC
- removed net D: 7SEG1.D, 7SEG2.D, U$2.SEGD
- removed net DIG0: 7SEG1.CC1, U$2.DIG0
- removed net DIG1: 7SEG1.CC2, U$2.DIG1
- removed net DIG2: 7SEG1.CC3, U$2.DIG2
- removed net DIG3: 7SEG1.CC4, U$2.DIG3
- removed net DIG4: 7SEG2.CC1, U$2.DIG4
- removed net DIG5: 7SEG2.CC2, U$2.DIG5
- removed net DIG6: 7SEG2.CC3, U$2.DIG6
- removed net DIG7: 7SEG2.CC4, U$2.DIG7
- removed net DP: 7SEG1.DP, 7SEG2.DP, U$2.SEGDP
- removed net E: 7SEG1.E, 7SEG2.E, U$2.SEGE
- removed net F: 7SEG1.F, 7SEG2.F, U$2.SEGF
- removed net G: 7SEG1.G, 7SEG2.G, U$2.SEGG
- removed net MAX_ISET: R1.1, U$2.ISET
- removed net N$1: JP2.1, JP2.2, U$1.OUT+
- removed net N$8: JP2.3, JP2.4, U$1.OUT-
- new net MATRIX_GND: JP4.4, U$1.OUT-
- new net MATRIX_VCC: JP4.1, U$1.OUT+
- net 5V: now also JP2.1, JP3.1; no longer C1.1, J1.4, J2.4, J3.4, J4.4, R1.2, U$2.VCC
- net CLK: now also JP2.3; no longer J1.2, J2.2, J3.2, J4.2
- net MAX_CLK: now also JP3.3; no longer U$2.CLK
- net MAX_DIN: now also JP3.5; no longer U$2.DIN
- net MAX_LOAD: now also JP3.4; no longer U$2.LOAD
- net MEGA_GND: now also JP2.2, JP3.2; no longer C1.2, J1.5, J2.5, J3.5, J4.5, U$2.GND@1, U$2.GND@2
- net PL: now also JP2.4; no longer J1.1, J2.1, J3.1, J4.1
- net SER1: now also JP2.8; no longer J4.3
- net SER2: now also JP2.7; no longer J3.3
- net SER3: now also JP2.6; no longer J2.3
- net SER4: now also JP2.5; no longer J1.3
Other:
- moved on the sheet: JP1, R2, X1-1, X1-2, X2-1, X2-10, X2-11, X2-12, X2-13, X2-14, X2-15, X2-16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
