File: Eagle_Verzeichnisse/Projekte/Matrix-Konsole/console1.brd (EAGLE design)
At the start: 43.2 x 130.5 mm, 5 parts, among them J1 DIN5, J2 DIN5, J3 DIN5, J4 DIN5

Commit message: Made final changes to the layout and added PDF-Files
Routing:
- net N$5: track 0.00 -> 348.0 mm
- net 5V: track 249.1 -> 250.6 mm
- net SER1: track 71.5 -> 72.6 mm
- net PL: track 166.5 -> 167.6 mm
- net MEGA_GND: track 154.4 -> 153.3 mm, vias 5 -> 6
- net SER4: track 57.6 -> 58.4 mm
- net CLK: track 195.2 -> 196.0 mm
