File: Eagle_Verzeichnisse/Projekte/Matrix-Konsole/console2.brd (EAGLE design)
At the start: 109.2 x 63.2 mm, 6 parts

Commit message: Made final changes to the layout and added PDF-Files
Routing:
- net N$5: track 0.00 -> 345.4 mm
- net DIG2: track 46.1 -> 36.7 mm
- net A: track 190.3 -> 198.7 mm
- net MEGA_GND: track 81.0 -> 73.7 mm
- net DIG0: track 86.0 -> 78.9 mm
- net MAX_CLK: track 51.5 -> 44.9 mm
- net 5V: track 75.6 -> 69.8 mm
- net DIG1: track 55.8 -> 50.2 mm
- net MAX_LOAD: track 42.5 -> 37.7 mm
- net B: track 88.4 -> 93.1 mm
- net DIG3: track 67.8 -> 72.1 mm
- net DIG6: track 76.0 -> 72.2 mm
- net C: track 88.8 -> 92.5 mm
- net DIG5: track 71.7 -> 68.3 mm
- net F: track 168.2 -> 165.2 mm
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